File: starbie.kicad_pcb (KiCad board)
At the start: 2 copper layers, 107.5 x 62.5 mm, 7 parts, among them J1 Conn_01x04_Pin, J3 Conn_01x08_Pin, SW1 SW_Push, SW2 SW_Push, U1 DHT11, U2 XIAO-ESP32-C3-SMD

Commit message: Update and add decal
Parts:
- added G***: LOGO, footprints:CubeBuddyLogov2, F.Cu at (144.5, 123.0)
Other:
- board size 107.5 x 62.5 mm -> 80 x 62.5 mm
